Commit message: added both wheel links

File: src/mobile_robot/model/mobile_robot.xacro (robot description, xacro)
@@ -1,29 +1,85 @@
-<?xml version = "1.0"?>
-<robot xmlns:xacro="https://www.ros.org/wiki/xacro" name = "mobile_robot">
-<link name="base_link">
-<visual>
-<geometry>
-<box size="0.30 0.20 0.10"/>
-</geometry>
-<material name = "blue">
-<color fgba="0 0 1 1"/>
-</material>
-</visual>
-<collision>
-<geometry>
-<box size="0.30 0.20 0.10"/>
-</geometry>
-</collision>
-<inertial>
-<mass value="2.0"/>
-<origin xyz="0 0 0"/>
-<inertia
-ixx="0.01"
-ixy="0"
-ixz="0"
-iyy="0.01"
-iyz="0"
-izz="0.02"/>
-</inertial>
-</link>
+<?xml version="1.0"?>
+<robot xmlns:xacro="https://www.ros.org/wiki/xacro" name="mobile_robot">
+    <link name="base_link">
+        <visual>
+            <geometry>
+                <box size="0.30 0.20 0.10" />
+            </geometry>
+            <material name="blue">
+                <color rgba="0 0 1 1" />
+            </material>
+        </visual>
+        <collision>
+            <geometry>
+                <box size="0.30 0.20 0.10" />
+            </geometry>
+        </collision>
+        <inertial>
+            <mass value="2.0" />
+            <origin xyz="0 0 0" />
+            <inertia
+                ixx="0.01"
+                ixy="0"
+                ixz="0"
+                iyy="0.01"
+                iyz="0"
+                izz="0.02" />
+        </inertial>
+    </link>
+    <link name="left_wheel">
+        <visual>
+            <geometry>
+                <cylinder radius="0.05" length="0.04"/>
+            </geometry>
+            <material name="black">
+                <color rgba="0 0 0 1"/>
+            </material>
+            <origin xyz="0 0 0" rpy="1.5708 0 0"/>
+        </visual>
+        <collision>
+            <geometry>
+                <cylinder raduis="0.05" length="0.04"/>
+            </geometry>
+            <origin xyz="0 0 0" rpy="1.5708 0 0"/>
+        </collision>
+        <inertial>
+            <mass value="0.2"/>
+            <origin xyz = "0 0 0"/>
+            <inertia
+            ixx = "0.0002"
+            ixy = "0"
+            ixz="0"
+            iyy="0.0002"
+            iyz="0"
+            izz="0.0001"/>
+        </inertial>
+    </link>
+    <link name="right_wheel">
+        <visual>
+            <geometry>
+                <cylinder radius="0.05" length="0.04"/>
+            </geometry>
+            <material name="black">
+                <color rgba="0 0 0 1"/>
+            </material>
+            <origin xyz="0 0 0" rpy="1.5708 0 0"/>
+        </visual>
+        <collision>
+            <geometry>
+                <cylinder raduis="0.05" length="0.04"/>
+            </geometry>
+            <origin xyz="0 0 0" rpy="1.5708 0 0"/>
+        </collision>
+        <inertial>
+            <mass value="0.2"/>
+            <origin xyz = "0 0 0"/>
+            <inertia
+            ixx = "0.0002"
+            ixy = "0"
+            ixz="0"
+            iyy="0.0002"
+            iyz="0"
+            izz="0.0001"/>
+        </inertial>
+    </link>
 </robot>

Commit message: Add continuous wheel joints

File: src/mobile_robot/model/mobile_robot.xacro (robot description, xacro)
@@ -39,5 +39,5 @@
         <collision>
             <geometry>
-                <cylinder raduis="0.05" length="0.04"/>
+                <cylinder radius="0.05" length="0.04"/>
             </geometry>
             <origin xyz="0 0 0" rpy="1.5708 0 0"/>
@@ -67,5 +67,5 @@
         <collision>
             <geometry>
-                <cylinder raduis="0.05" length="0.04"/>
+                <cylinder radius="0.05" length="0.04"/>
             </geometry>
             <origin xyz="0 0 0" rpy="1.5708 0 0"/>
@@ -83,3 +83,15 @@
         </inertial>
     </link>
+    <joint name="left_wheel_joint" type="continuous">
+        <parent link="base_link"/>
+        <child link="left_wheel"/>
+        <origin xyz="0 -0.12 -0.025" rpy="0 0 0"/>
+        <axis xyz="0 1 0"/>
+    </joint>
+    <joint name="right_wheel_joint" type="continuous">
+        <parent link="base_link"/>
+        <child link="right_wheel"/>
+        <origin xyz="0 -0.12 -0.025" rpy="0 0 0"/>
+        <axis xyz="0 1 0"/>
+    </joint>
 </robot>

Commit message: Fix robot visualization using Humble urdf_launch

File: src/mobile_robot/model/mobile_robot.xacro (robot description, xacro)
@@ -92,5 +92,5 @@
         <parent link="base_link"/>
         <child link="right_wheel"/>
-        <origin xyz="0 -0.12 -0.025" rpy="0 0 0"/>
+        <origin xyz="0 0.12 -0.025" rpy="0 0 0"/>
         <axis xyz="0 1 0"/>
     </joint>

Commit message: add gazebo stimulation code

File: src/mobile_robot/model/mobile_robot.xacro (robot description, xacro)
@@ -1,4 +1,5 @@
 <?xml version="1.0"?>
 <robot xmlns:xacro="https://www.ros.org/wiki/xacro" name="mobile_robot">
+    <xacro:include filename="$(find mobile_robot)/model/mobile_robot.gazebo" />
     <link name="base_link">
         <visual>
@@ -30,27 +31,27 @@
         <visual>
             <geometry>
-                <cylinder radius="0.05" length="0.04"/>
+                <cylinder radius="0.05" length="0.04" />
             </geometry>
             <material name="black">
-                <color rgba="0 0 0 1"/>
+                <color rgba="0 0 0 1" />
             </material>
-            <origin xyz="0 0 0" rpy="1.5708 0 0"/>
+            <origin xyz="0 0 0" rpy="1.5708 0 0" />
         </visual>
         <collision>
             <geometry>
-                <cylinder radius="0.05" length="0.04"/>
+                <cylinder radius="0.05" length="0.04" />
             </geometry>
-            <origin xyz="0 0 0" rpy="1.5708 0 0"/>
+            <origin xyz="0 0 0" rpy="1.5708 0 0" />
         </collision>
         <inertial>
-            <mass value="0.2"/>
-            <origin xyz = "0 0 0"/>
+            <mass value="0.2" />
+            <origin xyz="0 0 0" />
             <inertia
-            ixx = "0.0002"
-            ixy = "0"
-            ixz="0"
-            iyy="0.0002"
-            iyz="0"
-            izz="0.0001"/>
+                ixx="0.0002"
+                ixy="0"
+                ixz="0"
+                iyy="0.0002"
+                iyz="0"
+                izz="0.0001" />
         </inertial>
     </link>
@@ -58,40 +59,71 @@
         <visual>
             <geometry>
-                <cylinder radius="0.05" length="0.04"/>
+                <cylinder radius="0.05" length="0.04" />
             </geometry>
             <material name="black">
-                <color rgba="0 0 0 1"/>
+                <color rgba="0 0 0 1" />
             </material>
-            <origin xyz="0 0 0" rpy="1.5708 0 0"/>
+            <origin xyz="0 0 0" rpy="1.5708 0 0" />
         </visual>
         <collision>
             <geometry>
-                <cylinder radius="0.05" length="0.04"/>
+                <cylinder radius="0.05" length="0.04" />
             </geometry>
-            <origin xyz="0 0 0" rpy="1.5708 0 0"/>
+            <origin xyz="0 0 0" rpy="1.5708 0 0" />
         </collision>
         <inertial>
-            <mass value="0.2"/>
-            <origin xyz = "0 0 0"/>
+            <mass value="0.2" />
+            <origin xyz="0 0 0" />
             <inertia
-            ixx = "0.0002"
-            ixy = "0"
-            ixz="0"
-            iyy="0.0002"
-            iyz="0"
-            izz="0.0001"/>
+                ixx="0.0002"
+                ixy="0"
+                ixz="0"
+                iyy="0.0002"
+                iyz="0"
+                izz="0.0001" />
+        </inertial>
+    </link>
+    <joint name="lidar_joint" type="fixed">
+        <parent link="base_link" />
+        <child link="lidar_link" />
+        <origin xyz="0 0 0.08" rpy="0 0 0" />
+    </joint>
+    <link name="lidar_link">
+        <visual>
+            <origin xyz="0 0 0" />
+            <geometry>
+                <cylinder radius="0.03" length="0.04" />
+            </geometry>
+            <material name="black" />
+        </visual>
+        <collision>
+            <origin xyz="0 0 0" />
+            <geometry>
+                <cylinder radius="0.03" length="0.04" />
+            </geometry>
+        </collision>
+        <inertial>
+            <mass value="0.1" />
+            <origin xyz="0 0 0" />
+            <inertia
+                ixx="0.0001"
+                ixy="0"
+                ixz="0"
+                iyy="0.0001"
+                iyz="0"
+                izz="0.0001" />
         </inertial>
     </link>
     <joint name="left_wheel_joint" type="continuous">
-        <parent link="base_link"/>
-        <child link="left_wheel"/>
-        <origin xyz="0 -0.12 -0.025" rpy="0 0 0"/>
-        <axis xyz="0 1 0"/>
+        <parent link="base_link" />
+        <child link="left_wheel" />
+        <origin xyz="0 -0.12 -0.025" rpy="0 0 0" />
+        <axis xyz="0 1 0" />
     </joint>
     <joint name="right_wheel_joint" type="continuous">
-        <parent link="base_link"/>
-        <child link="right_wheel"/>
-        <origin xyz="0 0.12 -0.025" rpy="0 0 0"/>
-        <axis xyz="0 1 0"/>
+        <parent link="base_link" />
+        <child link="right_wheel" />
+        <origin xyz="0 0.12 -0.025" rpy="0 0 0" />
+        <axis xyz="0 1 0" />
     </joint>
 </robot>
